Commit message: change direction of axis in urdf

File: model/decopin_hand.urdf (robot description, URDF)
Before this commit: robot decopin_hand, 9 links, 8 joints
Joints:
- joint fixed_finger_middle_joint: axis 0 1 0 -> 0 -1 0
- joint fixed_finger_tip_joint: mimic (none) -> joint=fixed_finger_middle_joint multiplier=-1 offset=0
- joint rotated_finger_left_joint: axis 0 1 0 -> 0 -1 0
- joint rotated_finger_left_middle_joint: axis 0 1 0 -> 0 -1 0
- joint rotated_finger_left_tip_joint: mimic (none) -> joint=rotated_finger_left_middle_joint multiplier=-1 offset=0
- joint rotated_finger_right_joint: mimic joint=rotated_finger_left_joint multiplier=-1 offset=0 -> joint=rotated_finger_left_joint multiplier=1 offset=0
- joint rotated_finger_right_middle_joint: axis 0 1 0 -> 0 -1 0
- joint rotated_finger_right_tip_joint: mimic (none) -> joint=rotated_finger_right_middle_joint multiplier=-1 offset=0

Commit message: change direction of joint according to real dyanmixel placement

File: model/decopin_hand.urdf (robot description, URDF)
Before this commit: robot decopin_hand, 9 links, 8 joints
Joints:
- joint rotated_finger_left_joint: axis 0 -1 0 -> 0 1 0
- joint rotated_finger_right_middle_joint: axis 0 -1 0 -> 0 1 0

Commit message: fix bug in urdf axis direction

File: model/decopin_hand.urdf (robot description, URDF)
Before this commit: robot decopin_hand, 9 links, 8 joints
Joints:
- joint rotated_finger_right_joint: mimic joint=rotated_finger_left_joint multiplier=1 offset=0 -> joint=rotated_finger_left_joint multiplier=-1 offset=0

Commit message: increase velocity limit of joints

File: model/decopin_hand.urdf (robot description, URDF)
Before this commit: robot decopin_hand, 9 links, 8 joints
Joints:
- joint fixed_finger_middle_joint: limit (none) -> effort=30 velocity=3.1416
- joint fixed_finger_tip_joint: limit (none) -> effort=30 velocity=3.1416
- joint rotated_finger_left_joint: limit (none) -> effort=30 velocity=3.1416
- joint rotated_finger_left_middle_joint: limit (none) -> effort=30 velocity=3.1416
- joint rotated_finger_left_tip_joint: limit (none) -> effort=30 velocity=3.1416
- joint rotated_finger_right_joint: limit (none) -> effort=30 velocity=3.1416
- joint rotated_finger_right_middle_joint: limit (none) -> effort=30 velocity=3.1416
- joint rotated_finger_right_tip_joint: limit (none) -> effort=30 velocity=3.1416
